File: stenopcb.sch (KiCad schematic (older format))
At the start: 71 parts, among them K1 MAIN_RIGHT_TO_VOWELS_RIGHT, K2 MAIN_LEFT_TO_VOWELS_LEFT, K3 VOWELS_RIGHT_IN, K4 VOWELS_LEFT_IN, P1 MAIN_RIGHT_IN, P2 MAIN_RIGHT_TO_MAIN_LEFT, P3 MAIN_LEFT_IN, SW1 SPST, SW10 SPST, SW11 SPST, SW12 SPST, SW13 SPST, SW14 SPST, SW15 SPST, SW16 SPST, SW17 SPST, SW18 SPST, SW19 SPST, SW2 SPST, SW20 SPST, SW21 SPST, SW22 SPST, SW23 SPST, SW24 SPST, SW25 SPST, SW26 SPST, SW27 SPST, SW28 SPST, SW29 SPST, SW3 SPST, SW30 SPST, SW4 SPST, SW5 SPST, SW6 SPST, SW7 SPST, SW8 SPST, SW9 SPST

Commit message: my changes.. don't remember for what anymore :/
Parts:
- D25, D26: symbol LED -> LED-RESCUE-stenopcb
- R1, R2: symbol R -> R-RESCUE-stenopcb
Changed lines of the file:
@@
 EESchema Schematic File Version 2
+LIBS:stenopcb-rescue
 LIBS:power
 LIBS:device
@@
 LIBS:memory
 LIBS:xilinx
-LIBS:special
 LIBS:microcontrollers
 LIBS:dsp
@@
 LIBS:valves
 LIBS:stenopcb-cache
-EELAYER 27 0
+EELAYER 25 0
 EELAYER END
 $Descr A4 11693 8268
@@
 L_COL_4
 $Comp
-L R R1
+L R-RESCUE-stenopcb R1
 U 1 1 5227330E
 P 1850 1250
@@
 $EndComp
 $Comp
-L LED D25
+L LED-RESCUE-stenopcb D25
 U 1 1 52273328
 P 1850 1700
@@
 LED
 $Comp
-L R R2
+L R-RESCUE-stenopcb R2
 U 1 1 5227334E
 P 2100 5250
@@
 $EndComp
 $Comp
-L LED D26
+L LED-RESCUE-stenopcb D26
 U 1 1 52273354
 P 2100 5700
@@
 Text Label 4550 5950 0    60   ~ 0
 L_ROW_2
+Wire Notes Line
+	800  4250 6950 4250
+Wire Notes Line
+	6950 4250 6950 7650
+Wire Notes Line
+	6950 7650 800  7650
+Wire Notes Line
+	800  7650 800  4250
 $EndSCHEMATC
